File: 0014_GPS_Module_L86.kicad_sch (KiCad schematic)
At the start: 12 parts, among them J1 20279-001E-01, Q1 DTC143Z, Q2 DTC143Z, U1 L86-M33

Commit message: Add files via upload
Parts:
- added D3: LED, LED_SMD:LED_0603_1608Metric, symbol Device:LED
- added R5: 470r, Resistor_SMD:R_0603_1608Metric, symbol Device:R
- added U2: ~, Moduler_:pin_header, symbol moduler_pin:air
- C2: footprint (none) -> Capacitor_Tantalum_SMD:CP_EIA-2012-12_Kemet-R
- C3: footprint (none) -> Capacitor_SMD:C_0603_1608Metric
- D1, D2: footprint (none) -> LED_SMD:LED_0603_1608Metric
- J1: footprint IPEX_20279-001E-01 -> L-KLS1-IPEX-20279-001E-0:L-KLS1-IPEX-20279-001E-0
- Q1, Q2: footprint (none) -> Package_TO_SOT_SMD:SOT-323_SC-70
- R1, R2, R3, R4: footprint (none) -> Resistor_SMD:R_0603_1608Metric
- U1: footprint XCVR_L86-M33 -> L86:XCVR_L86-M33
Connections:
- net +3V3: now also R5.2, U2.8
- net FORCE_ON: now also U2.13
- net GND: now also D3.1 (K), U2.9
- net RESET: now also U2.12
- net RX: now also U2.11
- net TX: now also U2.10
- new net: D3.2 (A), R5.1
- no-connect marks 1 -> 13
Other:
- note added: "AIR PIN"
- note added: "SENSOR"
- moved on the sheet: C2, C3, D1, D2, J1, Q1, Q2, R1, R2, R3, R4, U1
